File: KiCad/ugv-robot/ugv-robot.kicad_sch (KiCad schematic)
At the start: 18 parts, among them J1 Charging_Port, SW1 LRF, SW2 Zoom_In, SW3 Zoom_Out, SW4 Body_Up, SW5 Body_Down, SW6 Lamp, U1 Analog_Joystick, U10 RF_MHz, U2 Digital_Joystick, U3 Boost_Conv, U4 Asus_NUC, U6 Monitor, U7 USB_HUB, U8 Keyboard_Mouse, U9 RF_GHz

Commit message: Reorganize project into Rapih/ folder structure
Move final Arduino, GCS app, and STM32 firmware source into Rapih/Code/,
and datasheets/schematics into Rapih/Datasheet/ and Rapih/Schematic/,
consolidating scattered old locations (gcs_app/, STM32Cube/motorugv_G474RE/,
Testcode/megapro_gcs/, Hardware/STM32G474_Board/) for a cleaner layout.
Other:
- company: (none) -> PT Respati Solusi Rekatama
- title: (none) -> UGV Robot
Changed lines of the file:
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@@
 	(generator_version "10.0")
 	(paper "A4")
+	(title_block
+		(title "UGV Robot")
+		(date "2026-08-03")
+		(rev "1")
+		(company "PT Respati Solusi Rekatama")
+		(comment 1 "Arduino Mega Pro")
+		(comment 2 "Asus NUC")
+		(comment 3 "GCS Schematic")
+		(comment 4 "UGV Project")
+		(comment 5 "5")
+		(comment 6 "6")
+		(comment 7 "7")
+		(comment 8 "8")
+		(comment 9 "9")
+	)
 	(rectangle
 		(start 116.84 13.97)
