File: Hardware/STM32G474/STM32G474.kicad_sch (KiCad schematic)
At the start: 0 parts

Commit message: Update STM32G474 schematic with MCU and USB buck sheets
Co-Authored-By: Claude Sonnet 5 <noreply@anthropic.com>
Other:
- added sheet MCU (MCU_sch.kicad_sch)
- added sheet USB & Buck (usbbuck_sch.kicad_sch)
