File: Hardware/STM32G474_Board/STM32G474_Board/STM32G474_Board.kicad_pcb (KiCad board)
At the start: 2 copper layers, 100 x 130 mm, 21 parts, among them CN1 NUCLEO (STM32G474RET6), J1 Steer_FL, J10 Jetson, J11 RF, J12 RS485, J13 Lamp_F, J14 Lamp_B, J15 Motor_FL, J16 Motor_BL, J17 Motor_FR, J18 Motor_BR, J19 Power, J2 Steer_BL, J3 Steer_FR, J4 Steer_BR, J5 Body_FL, J6 Body_BL, J7 Body_FR, J8 Body_BR, J9 Debug

Commit message: firmware
Connections:
- CN1 pad 27: LinearL_3 -> unconnected-(CN1-PC15-Pad27)
- CN1 pad 29: LinearR_3 -> unconnected-(CN1-PF0-Pad29)
- CN1 pad 31: LinearL_5 -> unconnected-(CN1-PF1-Pad31)
- CN1 pad 32: unconnected-(CN1-PA4-Pad32) -> LinearL_5
- CN1 pad 54: unconnected-(CN1-PB12-Pad54) -> LinearL_3
- CN1 pad 68: unconnected-(CN1-PB13-Pad68) -> LinearR_3
Routing:
- net LinearR_3: track 50.0 -> 165.1 mm, vias 0 -> 2
- net LinearL_3: track 49.9 -> 140.5 mm, vias 0 -> 2
- net LinearL_5: track 60.2 -> 94.8 mm, vias 0 -> 1
- net Lamp_F: track 91.5 -> 95.9 mm
- net Lamp_B: track 83.8 -> 87.8 mm
- net MotorS_1: track 104.1 -> 107.8 mm
- net MotorP_1: track 114.0 -> 117.6 mm
- net +5V: track 269.5 -> 270.8 mm
- net MotorP_3: track 145.0 -> 145.5 mm
- net Jetson_RX: track 112.5 -> 113.0 mm
