File: Hardware/STM32G474_Board/STM32G474_Board/STM32G474_Board.kicad_sch (KiCad schematic)
At the start: 20 parts, among them CN1 NUCLEO (STM32G474RET6), J1 Steer_FL, J10 Jetson, J11 RF, J12 RS485, J13 Lamp_F, J14 Lamp_B, J15 Motor_FL, J16 Motor_BL, J17 Motor_FR, J18 Motor_BR, J19 Power, J2 Steer_BL, J3 Steer_FR, J4 Steer_BR, J5 Body_FL, J6 Body_BL, J7 Body_FR, J8 Body_BR, J9 Debug

Commit message: Firmware
Parts:
- removed J10: Jetson, Connector_JST:JST_XH_B2B-XH-A_1x02_P2.50mm_Vertical, symbol Connector:Conn_01x02_Pin
- removed J13: Lamp_F, Connector_JST:JST_XH_B3B-XH-A_1x03_P2.50mm_Vertical, symbol Connector:Conn_01x03_Pin
- removed J14: Lamp_B, Connector_JST:JST_XH_B3B-XH-A_1x03_P2.50mm_Vertical, symbol Connector:Conn_01x03_Pin
- removed J9: Debug, Connector_JST:JST_XH_B2B-XH-A_1x02_P2.50mm_Vertical, symbol Connector:Conn_01x02_Pin
- added J10: Jetson, Connector_JST:JST_XH_B3B-XH-A_1x03_P2.50mm_Vertical, symbol Connector:Conn_01x03_Pin
- added J13: Lamp_F, Connector_JST:JST_XH_B4B-XH-A_1x04_P2.50mm_Vertical, symbol Connector:Conn_01x04_Pin
- added J14: Lamp_B, Connector_JST:JST_XH_B4B-XH-A_1x04_P2.50mm_Vertical, symbol Connector:Conn_01x04_Pin
- added J9: Debug, Connector_JST:JST_XH_B3B-XH-A_1x03_P2.50mm_Vertical, symbol Connector:Conn_01x03_Pin
- J1, J11, J12, J15, J16, J17, J18, J19, J2, J3, J4, J5, J6, J7, J8: KiLib_Generator (none) -> connector/JST
Connections:
- net +5V: now also CN1.6 (E5V), J13.1 (Pin_1), J14.1 (Pin_1); no longer CN1.24 (VIN)
- net Debug_RX: now also J9.2 (Pin_2)
- net Debug_TX: now also J9.1 (Pin_1)
- net GND: now also J10.3 (Pin_3), J13.4 (Pin_4), J14.4 (Pin_4), J9.3 (Pin_3)
- net Jetson_RX: now also J10.2 (Pin_2)
- net Jetson_TX: now also J10.1 (Pin_1)
- net Lamp_B: now also J14.3 (Pin_3)
- net Lamp_F: now also J13.3 (Pin_3)
- net LinearL_0: now also CN1.4 (PD2); no longer CN1.25 (PC14)
- net LinearL_1: now also CN1.53 (PA7); no longer CN1.57 (PC7)
- net LinearL_2: now also CN1.30 (PA1); no longer CN1.39 (PC9)
- net LinearL_3: now also CN1.27 (PC15); no longer CN1.2 (PC11)
- net LinearL_4: now also CN1.1 (PC10); no longer CN1.29 (PF0)
- net LinearL_5: now also CN1.31 (PF1); no longer CN1.49 (PA5)
- net LinearL_7: now also CN1.59 (PA9); no longer CN1.71 (PA10)
- net LinearR_0: now also CN1.2 (PC11); no longer CN1.23 (PC13)
- net LinearR_1: now also CN1.39 (PC9); no longer CN1.27 (PC15)
- net LinearR_2: now also CN1.28 (PA0); no longer CN1.40 (PC8)
- net LinearR_3: now also CN1.29 (PF0); no longer CN1.1 (PC10)
- net LinearR_5: now also CN1.35 (PC2); no longer CN1.31 (PF1)
- net LinearR_6: now also CN1.71 (PA10); no longer CN1.53 (PA7)
- net LinearR_7: now also CN1.57 (PC7); no longer CN1.59 (PA9)
- net MotorS_0: now also CN1.49 (PA5); no longer CN1.28 (PA0)
- net MotorS_1: now also CN1.23 (PC13); no longer CN1.30 (PA1)
- net MotorS_2: now also CN1.40 (PC8); no longer CN1.35 (PC2)
- net T_SWCLK: no longer names the net of CN1.15 (PA14)
- net T_SWDIO: no longer names the net of CN1.13 (PA13)
- no-connect marks 36 -> 40
Other:
- company: (none) -> PT Respati Solusi Rekatama
- title: (none) -> STM32G474RE Board - UGV
- moved on the sheet: CN1, J1, J11, J12, J15, J16, J17, J18, J19, J2, J3, J4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

Commit message: firmware
Connections:
- net LinearL_3: now also CN1.54 (PB12); no longer CN1.27 (PC15)
- net LinearL_5: now also CN1.32 (PA4); no longer CN1.31 (PF1)
- net LinearR_3: now also CN1.68 (PB13); no longer CN1.29 (PF0)
